File: MMS3/VRM.kicad_sch (KiCad schematic)
At the start: 0 parts

Commit message: schematic + partly layout
Parts:
- added C30, C31, C32, C33, C34, C35: 10uF, PCM_JLCPCB:C_0805, symbol PCM_JLCPCB-Capacitors:0805,10uF,(2)
- added C38, C39: 220nF, PCM_JLCPCB:C_0805, symbol PCM_JLCPCB-Capacitors:0805,220nF
- added C40: 100nF, PCM_JLCPCB:C_0805, symbol PCM_JLCPCB-Capacitors:0805,100nF
- added C41, C42, C45, C46, C47: 22uF, PCM_JLCPCB:C_0805, symbol PCM_JLCPCB-Capacitors:0805,22uF
- added C43: 47pF, PCM_JLCPCB:C_0402, symbol PCM_JLCPCB-Capacitors:0402,47pF
- added C44: 4.7nF, PCM_JLCPCB:C_0402, symbol PCM_JLCPCB-Capacitors:0402,4.7nF
- added C49, C50: 100uF, Capacitor_SMD:CP_Elec_10x10, symbol Device:C_Polarized
- added C69, C74: 100nF, PCM_JLCPCB:C_0402, symbol PCM_JLCPCB-Capacitors:0402,100nF
- added D1: SMF58CA, PCM_JLCPCB:D_SOD-123FL, symbol PCM_JLCPCB-Diodes:TVS-Uni,SMF58CA
- added D3, D4: SS510B, PCM_JLCPCB:D_SMB, symbol PCM_JLCPCB-Diodes:Schottky,SS510B
- added L1: YSPI1050-100M, Inductor_SMD:L_Sunlord_MWSA1005S, symbol Device:L
- added R33, R34: 24.9kΩ, PCM_JLCPCB:R_0402, symbol PCM_JLCPCB-Resistors:0402,24kΩ
- added R36: 43kΩ, PCM_JLCPCB:R_0603, symbol PCM_JLCPCB-Resistors:0603,43kΩ
- added R37: 8.2kΩ, PCM_JLCPCB:R_0402, symbol PCM_JLCPCB-Resistors:0402,8.2kΩ
- added R38: 12kΩ, PCM_JLCPCB:R_0402, symbol PCM_JLCPCB-Resistors:0402,12kΩ
- added R39: 240kΩ, PCM_JLCPCB:R_0603, symbol PCM_JLCPCB-Resistors:0603,240kΩ
- added TP16, TP17, TP18, TP19, TP20: TestPoint, TestPoint:TestPoint_Pad_D1.0mm, symbol Connector:TestPoint
- added U15: AMS1117-3.3, Package_TO_SOT_SMD:SOT-223-3_TabPin2, symbol Regulator_Linear:AMS1117-3.3
- added U2: TPS54560BDDA, Package_SO:Texas_R-PDSO-G8_EP2.95x4.9mm_Mask2.4x3.1mm_ThermalVias, symbol Regulator_Switching:TPS54560BDDA
Connections:
- new net: C41.1, C42.1, C45.1, C46.1, C47.1, D4.2, L1.2, R36.1, TP19.1
- new net: C43.1, R38.1, TP17.1, U2.6 (COMP)
- new net: R39.1, TP20.1, U2.4 (RT/CLK)
- new net: R36.2, R37.1, TP18.1, U2.5 (FB)
- new net: C40.1, D3.1, L1.1, U2.8 (SW)
- new net: C40.2, U2.1 (BOOT)
- new net: C44.1, R38.2
- new net +3V3: C69.1, U15.2 (VO)
- new net +5V: C50.1, C74.1, D4.1, U15.3 (VI)
- new net Cap_protec: C30.2, C31.1, C32.2, C33.1, C34.2, C35.1, C38.2, C39.1, R33.2, R34.1
- new net GND: C31.2, C33.2, C35.2, C39.2, C41.2, C42.2, C43.2, C44.2, C45.2, C46.2, C47.2, C49.2, C50.2, C69.2, C74.2, D1.2, D3.2, R34.2, R37.2, R39.2, U15.1 (GND), U2.7 (GND), U2.9 (GND)
- new net Vin: C30.1, C32.1, C34.1, C38.1, C49.1, D1.1, R33.1, TP16.1, U2.2 (VIN), U2.3 (EN)
Other:
- note added: "60V MAX"
- note added: "IEC 60664-1 Material Group III (CTI < 400; typical FR-4 = IIIa): 1.25 mm"
- note added: "INFORMATION"
- note added: "KEEP CRIPPAGE DISTANCE 1.26MM MIN!"
- note added: "RANDOM NUMBER GENERATOR OUTPUT"
- note added: "Thats not sketch ... thats BOM-bastic!"
- note added: "saved for kebab on that one alone"
