File: MMS3/VRM.kicad_sch (KiCad schematic)
At the start: 37 parts, among them U15 AMS1117-3.3, U2 TPS54560BDDA

Commit message: prod ready
Other:
- moved on the sheet: C49
Changed lines of the file:
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@@
 	)
 	(junction
-		(at 91.44 152.4)
+		(at 88.9 152.4)
 		(diameter 0)
 		(color 0 0 0 0)
@@
 	)
 	(junction
+		(at 88.9 129.54)
+		(diameter 0)
+		(color 0 0 0 0)
+	)
+	(junction
 		(at 100.33 152.4)
 		(diameter 0)
@@
 	)
 	(junction
-		(at 91.44 129.54)
+		(at 254 134.62)
 		(diameter 0)
 		(color 0 0 0 0)
 	)
 	(junction
-		(at 254 134.62)
+		(at 241.3 81.28)
+		(diameter 0)
+		(color 0 0 0 0)
+	)
+	(junction
+		(at 186.69 129.54)
 		(diameter 0)
 		(color 0 0 0 0)
@@
 	(wire
 		(pts
+			(xy 88.9 152.4) (xy 100.33 152.4)
+		)
+		(stroke
+			(width 0)
+			(type default)
+		)
+	)
+	(wire
+		(pts
 			(xy 285.75 134.62) (xy 299.72 134.62)
 		)
@@
 	(wire
 		(pts
-			(xy 91.44 146.05) (xy 91.44 152.4)
+			(xy 88.9 146.05) (xy 88.9 152.4)
 		)
 		(stroke
@@
 	(wire
 		(pts
+			(xy 241.3 81.28) (xy 238.76 81.28)
+		)
+		(stroke
+			(width 0)
+			(type default)
+		)
+	)
+	(wire
+		(pts
+			(xy 88.9 129.54) (xy 100.33 129.54)
+		)
+		(stroke
+			(width 0)
+			(type default)
+		)
+	)
+	(wire
+		(pts
 			(xy 170.18 142.24) (xy 176.53 142.24)
 		)
@@
 	(wire
 		(pts
-			(xy 91.44 129.54) (xy 91.44 138.43)
+			(xy 88.9 129.54) (xy 88.9 138.43)
 		)
 		(stroke
@@
 	(wire
 		(pts
-			(xy 77.47 129.54) (xy 91.44 129.54)
+			(xy 77.47 129.54) (xy 88.9 129.54)
 		)
 		(stroke
@@
 	(wire
 		(pts
-			(xy 77.47 152.4) (xy 91.44 152.4)
+			(xy 77.47 152.4) (xy 88.9 152.4)
 		)
 		(stroke
@@
 	(wire
 		(pts
-			(xy 160.02 129.54) (xy 193.04 129.54)
-		)
-		(stroke
-			(width 0)
-			(type default)
-		)
-	)
-	(wire
-		(pts
-			(xy 91.44 152.4) (xy 100.33 152.4)
+			(xy 160.02 129.54) (xy 186.69 129.54)
 		)
 		(stroke
@@
 	(wire
 		(pts
-			(xy 91.44 129.54) (xy 100.33 129.54)
-		)
-		(stroke
-			(width 0)
-			(type default)
-		)
-	)
-	(wire
-		(pts
 			(xy 261.62 134.62) (xy 261.62 142.24)
 		)
@@
 	(wire
 		(pts
+			(xy 186.69 129.54) (xy 193.04 129.54)
+		)
+		(stroke
+			(width 0)
+			(type default)
+		)
+	)
+	(wire
+		(pts
 			(xy 132.08 129.54) (xy 152.4 129.54)
 		)
@@
 	(wire
 		(pts
-			(xy 246.38 81.28) (xy 238.76 81.28)
+			(xy 246.38 81.28) (xy 241.3 81.28)
 		)
 		(stroke
@@
 	)
 	(symbol
+		(lib_id "power:PWR_FLAG")
+		(at 241.3 81.28 0)
+		(unit 1)
+		(body_style 1)
+		(exclude_from_sim no)
+		(in_bom yes)
+		(on_board yes)
+		(in_pos_files yes)
+		(dnp no)
+		(fields_autoplaced yes)
+		(property "Reference" "#FLG04"
+			(at 241.3 79.375 0)
+			(hide yes)
+			(show_name no)
+			(do_not_autoplace no)
+			(effects
+				(font
+					(size 1.27 1.27)
+				)
+			)
+		)
+		(property "Value" "PWR_FLAG"
+			(at 241.3 76.2 0)
+			(show_name no)
+			(do_not_autoplace no)
+			(effects
+				(font
+					(size 1.27 1.27)
+				)
+			)
+		)
+		(property "Footprint" ""
+			(at 241.3 81.28 0)
+			(hide yes)
+			(show_name no)
+			(do_not_autoplace no)
+			(effects
+				(font
+					(size 1.27 1.27)
+				)
+			)
+		)
+		(property "Datasheet" ""
+			(at 241.3 81.28 0)
+			(hide yes)
+			(show_name no)
+			(do_not_autoplace no)
+			(effects
+				(font
+					(size 1.27 1.27)
+				)
+			)
+		)
+		(property "Description" "Special symbol for telling ERC where power comes from"
+			(at 241.3 81.28 0)
+			(hide yes)
+			(show_name no)
+			(do_not_autoplace no)
+			(effects
+				(font
+					(size 1.27 1.27)
+				)
+			)
+		)
+		(pin "1"
+		)
+		(instances
+			(project "MMS3"
+				(path "/712cea22-140d-4c92-923f-f4998caf3ecd/86aabed7-d22c-4284-aa19-8f20b4664afb"
+					(reference "#FLG04")
+					(unit 1)
+				)
+			)
+		)
+	)
+	(symbol
 		(lib_id "PCM_JLCPCB-Capacitors:0805,22uF")
 		(at 276.86 146.05 0)
@@
 	)
 	(symbol
+		(lib_id "power:PWR_FLAG")
+		(at 186.69 129.54 0)
+		(unit 1)
+		(body_style 1)
+		(exclude_from_sim no)
+		(in_bom yes)
+		(on_board yes)
+		(in_pos_files yes)
+		(dnp no)
+		(fields_autoplaced yes)
+		(property "Reference" "#FLG03"
+			(at 186.69 127.635 0)
+			(hide yes)
+			(show_name no)
+			(do_not_autoplace no)
+			(effects
+				(font
+					(size 1.27 1.27)
+				)
+			)
+		)
+		(property "Value" "PWR_FLAG"
+			(at 186.69 124.46 0)
+			(show_name no)
+			(do_not_autoplace no)
+			(effects
+				(font
+					(size 1.27 1.27)
+				)
+			)
+		)
+		(property "Footprint" ""
+			(at 186.69 129.54 0)
+			(hide yes)
+			(show_name no)
+			(do_not_autoplace no)
+			(effects
+				(font
+					(size 1.27 1.27)
+				)
+			)
+		)
+		(property "Datasheet" ""
+			(at 186.69 129.54 0)
+			(hide yes)
+			(show_name no)
+			(do_not_autoplace no)
+			(effects
+				(font
+					(size 1.27 1.27)
+				)
+			)
+		)
+		(property "Description" "Special symbol for telling ERC where power comes from"
+			(at 186.69 129.54 0)
+			(hide yes)
+			(show_name no)
+			(do_not_autoplace no)
+			(effects
+				(font
+					(size 1.27 1.27)
+				)
+			)
+		)
+		(pin "1"
+		)
+		(instances
+			(project "MMS3"
+				(path "/712cea22-140d-4c92-923f-f4998caf3ecd/86aabed7-d22c-4284-aa19-8f20b4664afb"
+					(reference "#FLG03")
+					(unit 1)
+				)
+			)
+		)
+	)
+	(symbol
 		(lib_id "PCM_JLCPCB-Resistors:0402,8.2kΩ")
 		(at 299.72 153.67 0)
@@
 	(symbol
 		(lib_id "Device:C_Polarized")
-		(at 91.44 142.24 0)
+		(at 88.9 142.24 0)
 		(unit 1)
 		(body_style 1)
@@
 		(fields_autoplaced yes)
 		(property "Reference" "C49"
-			(at 95.25 140.0809 0)
+			(at 92.71 140.0809 0)
 			(show_name no)
 			(do_not_autoplace no)
@@
 		)
 		(property "Value" "100uF"
-			(at 95.25 142.6209 0)
+			(at 92.71 142.6209 0)
 			(show_name no)
 			(do_not_autoplace no)
@@
 		)
 		(property "Footprint" "Capacitor_SMD:CP_Elec_10x10"
-			(at 92.4052 146.05 0)
+			(at 89.8652 146.05 0)
 			(hide yes)
 			(show_name no)
@@
 		)
 		(property "Datasheet" ""
-			(at 91.44 142.24 0)
+			(at 88.9 142.24 0)
 			(hide yes)
 			(show_name no)
@@
 		)
 		(property "Description" "Polarized capacitor"
-			(at 91.44 142.24 0)
+			(at 88.9 142.24 0)
 			(hide yes)
 			(show_name no)
@@
 		)
 		(property "LCSC" "C249838"
-			(at 91.44 142.24 0)
+			(at 88.9 142.24 0)
 			(hide yes)
 			(show_name no)
@@
 		)
 		(property "MPN" "VZH101M1KTR-1010"
-			(at 91.44 142.24 0)
+			(at 88.9 142.24 0)
 			(hide yes)
 			(show_name no)
