File: MMS3/MCU.kicad_sch (KiCad schematic)
At the start: 35 parts, among them SW1 BOOT, SW2 RESET, U1 STM32F405RGTx, X1 X32258MOB4SI, X2 Q13FC1350000400

Commit message: schematic + partly layout
Parts:
- removed C12, C14: 10uF, PCM_JLCPCB:C_0603, symbol PCM_JLCPCB-Capacitors:0603,10uF
- removed SW1: BOOT, Button_Switch_SMD:SW_Tactile_SPST_NO_Straight_CK_PTS636Sx25SMTRLFS, symbol Switch:SW_Push
- removed SW2: RESET, Button_Switch_SMD:SW_Tactile_SPST_NO_Straight_CK_PTS636Sx25SMTRLFS, symbol Switch:SW_Push
- removed TP6: TestPoint, TestPoint:TestPoint_Pad_D1.0mm, symbol Connector:TestPoint
- added C12: 100nF, PCM_JLCPCB:C_0402, symbol PCM_JLCPCB-Capacitors:0402,100nF
- added C36, C37: 10uF, PCM_JLCPCB:C_0402, symbol PCM_JLCPCB-Capacitors:0402,10uF
- added LED1: FixLed307, FixLed307:FixLed307, symbol FixLed307:FixLed307
- added R22: 100Ω, PCM_JLCPCB:R_0402, symbol PCM_JLCPCB-Resistors:0402,100Ω
- added R27, R40: 1kΩ, PCM_JLCPCB:R_0402, symbol PCM_JLCPCB-Resistors:0402,1kΩ
- added SW3, SW5: TC-6615Z-12.5-260, Tact-sw:SW-TH_4P-L7.3-TC-6615Z-12.5-260, symbol Tact-sw:TC-6615Z-12.5-260
Connections:
- net +3V3: now also C37.1, R40.1
- net BOOT_EN: now also U1.20 (PA4)
- net GND: now also C12.2, C36.2, C37.2, LED1.2, LED1.4, SW3.2 (B), SW3.3 (C), SW3.4 (D), SW5.2 (B), SW5.3 (C), SW5.4 (D)
- net NRST: now also R22.1; no longer U1.7 (NRST)
- net SWD.~{RST}: now also SW3.1 (A)
- net USR_BUTTON: now also SW5.1 (A)
- net VDDA: now also C36.1
- net I2C_Memory_addr renamed USER_LED_3
- net USER_LED_3: now also R27.1
- new net: C12.1, R22.2, U1.7 (NRST)
- new net: LED1.3, R27.2
- new net: LED1.1, R40.2
- no-connect marks 2 -> 1
Other:
- note removed: "I2C MEME"
- moved on the sheet: C13, C15, C18, C25, C26, FB401, R10, R11, R12, R13, R14, R15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

Commit message: almost done
Connections:
- net NRST: no longer C26.1, R12.1, R15.1
- net Chainbus_I2C_addr0 renamed Chainbus.CS
- net Chainbus_I2C_addr1 renamed Chainbus_addr4
- net Chainbus_I2C_addr2 renamed Chainbus_addr3
- net Chainbus_SPI_CS0 renamed Chainbus_addr5
- net Chainbus_SPI_CS1 renamed Chainbus_addr6
- net Chainbus_SPI_CS2 renamed Chainbus_addr7
- net Chainbus_UART_addr0 renamed Chainbus_addr1
- net Chainbus_UART_addr1 renamed Chainbus_addr0
- net Chainbus_UART_addr2 renamed Chainbus_addr2
- new net: C26.1, R15.1
Other:
- note removed: "CHAINBUS I2C"
- note removed: "CHAINBUS SPI"
- note removed: "CHAINBUS UART"
- moved on the sheet: C10, C11, C13, C15, C18, C25, C26, C36, C37, C8, C9, FB401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
