File: MMS3/MCU.kicad_sch (KiCad schematic)
At the start: 39 parts, among them SW3 TC-6615Z-12.5-260, SW5 TC-6615Z-12.5-260, U1 STM32F405RGTx, X1 X32258MOB4SI, X2 Q13FC1350000400

Commit message: prod ready
Connections:
- net NRST: now also C26.1, R12.1, R15.1
- no-connect marks 1 -> 2
Changed lines of the file:
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@@
 	)
 	(junction
+		(at 55.88 231.14)
+		(diameter 0)
+		(color 0 0 0 0)
+	)
+	(junction
 		(at 308.61 111.76)
 		(diameter 0)
@@
 		(at 323.85 175.26)
 	)
+	(no_connect
+		(at 280.67 182.88)
+	)
 	(bus_entry
 		(at 481.33 196.85)
@@
 	(wire
 		(pts
+			(xy 53.34 231.14) (xy 55.88 231.14)
+		)
+		(stroke
+			(width 0)
+			(type default)
+		)
+	)
+	(wire
+		(pts
 			(xy 81.28 191.77) (xy 76.2 191.77)
 		)
@@
 	(wire
 		(pts
-			(xy 53.34 231.14) (xy 45.72 231.14)
-		)
-		(stroke
-			(width 0)
-			(type default)
-		)
-	)
-	(wire
-		(pts
 			(xy 273.05 162.56) (xy 283.21 162.56)
 		)
@@
 		)
 	)
+	(wire
+		(pts
+			(xy 280.67 182.88) (xy 283.21 182.88)
+		)
+		(stroke
+			(width 0)
+			(type default)
+		)
+	)
 	(bus
 		(pts
@@
 		)
 	)
+	(wire
+		(pts
+			(xy 55.88 231.14) (xy 60.96 231.14)
+		)
+		(stroke
+			(width 0)
+			(type default)
+		)
+	)
 	(bus
 		(pts
@@
 	(wire
 		(pts
+			(xy 55.88 228.6) (xy 55.88 231.14)
+		)
+		(stroke
+			(width 0)
+			(type default)
+		)
+	)
+	(wire
+		(pts
 			(xy 471.17 298.45) (xy 471.17 300.99)
 		)
@@
 	)
 	(label "NRST"
-		(at 54.61 231.14 0)
+		(at 55.88 228.6 0)
 		(effects
 			(font
