File: MMS3/Interboard_connector.kicad_sch (KiCad schematic)
At the start: 1 part, among them J1 86093488324755V1LF

Commit message: prod ready
Changed lines of the file:
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@@
 		)
 	)
+	(junction
+		(at 128.27 137.16)
+		(diameter 0)
+		(color 0 0 0 0)
+	)
 	(no_connect
 		(at 147.32 134.62)
@@
 		)
 	)
+	(wire
+		(pts
+			(xy 128.27 137.16) (xy 147.32 137.16)
+		)
+		(stroke
+			(width 0)
+			(type default)
+		)
+	)
 	(bus
 		(pts
@@
 	(wire
 		(pts
+			(xy 128.27 133.35) (xy 128.27 137.16)
+		)
+		(stroke
+			(width 0)
+			(type default)
+		)
+	)
+	(wire
+		(pts
 			(xy 177.8 73.66) (xy 207.01 73.66)
 		)
@@
 	(wire
 		(pts
-			(xy 144.78 137.16) (xy 147.32 137.16)
+			(xy 121.92 137.16) (xy 128.27 137.16)
 		)
 		(stroke
@@
 	)
 	(symbol
+		(lib_id "power:PWR_FLAG")
+		(at 128.27 133.35 0)
+		(unit 1)
+		(body_style 1)
+		(exclude_from_sim no)
+		(in_bom yes)
+		(on_board yes)
+		(in_pos_files yes)
+		(dnp no)
+		(fields_autoplaced yes)
+		(property "Reference" "#FLG05"
+			(at 128.27 131.445 0)
+			(hide yes)
+			(show_name no)
+			(do_not_autoplace no)
+			(effects
+				(font
+					(size 1.27 1.27)
+				)
+			)
+		)
+		(property "Value" "PWR_FLAG"
+			(at 128.27 128.27 0)
+			(show_name no)
+			(do_not_autoplace no)
+			(effects
+				(font
+					(size 1.27 1.27)
+				)
+			)
+		)
+		(property "Footprint" ""
+			(at 128.27 133.35 0)
+			(hide yes)
+			(show_name no)
+			(do_not_autoplace no)
+			(effects
+				(font
+					(size 1.27 1.27)
+				)
+			)
+		)
+		(property "Datasheet" ""
+			(at 128.27 133.35 0)
+			(hide yes)
+			(show_name no)
+			(do_not_autoplace no)
+			(effects
+				(font
+					(size 1.27 1.27)
+				)
+			)
+		)
+		(property "Description" "Special symbol for telling ERC where power comes from"
+			(at 128.27 133.35 0)
+			(hide yes)
+			(show_name no)
+			(do_not_autoplace no)
+			(effects
+				(font
+					(size 1.27 1.27)
+				)
+			)
+		)
+		(pin "1"
+		)
+		(instances
+			(project "MMS3"
+				(path "/712cea22-140d-4c92-923f-f4998caf3ecd/05cbb48a-06b7-415e-80f6-4593be6cf8dc"
+					(reference "#FLG05")
+					(unit 1)
+				)
+			)
+		)
+	)
+	(symbol
 		(lib_id "power:+5V")
-		(at 144.78 137.16 90)
+		(at 121.92 137.16 90)
 		(unit 1)
 		(body_style 1)
@@
 		(fields_autoplaced yes)
 		(property "Reference" "#PWR070"
-			(at 148.59 137.16 0)
+			(at 125.73 137.16 0)
 			(hide yes)
 			(show_name no)
@@
 		)
 		(property "Value" "+12V stby"
-			(at 140.97 137.1599 90)
+			(at 118.11 137.1599 90)
 			(show_name no)
 			(do_not_autoplace no)
@@
 		)
 		(property "Footprint" ""
-			(at 144.78 137.16 0)
+			(at 121.92 137.16 0)
 			(hide yes)
 			(show_name no)
@@
 		)
 		(property "Datasheet" ""
-			(at 144.78 137.16 0)
+			(at 121.92 137.16 0)
 			(hide yes)
 			(show_name no)
@@
 		)
 		(property "Description" "Power symbol creates a global label with name \"+5V\""
-			(at 144.78 137.16 0)
+			(at 121.92 137.16 0)
 			(hide yes)
 			(show_name no)
