File: MMS3/Slide-SW.kicad_sch (KiCad schematic)
At the start: 3 parts, among them SW4 SK12D07VG5

Commit message: prod ready
Connections:
- no-connect marks 0 -> 1
Changed lines of the file:
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@@
 		(color 0 0 0 0)
+	)
+	(no_connect
+		(at 106.68 97.79)
 	)
 	(wire
